File: EDA files/EEZ DIB MIO168 r2B4.sch (EAGLE design)
At the start: 302 parts, among them IC1 M24C32-WMN6P, IC10 DAC7760IPWPR, IC11 DAC7760IPWPR, IC12 OPA376AIDBVR, IC13 DAC7563TDGSR, IC14 OPA2196IDR, IC15 BTS3408G, IC16 BTS3408G, IC17 BTS3408G, IC18 BTS3408G, IC19 74HC126PW,118, IC2 Si8641BB-B-IS1, IC20 TL431B, IC21 DG468DV-T1-E3, IC22 DG468DV-T1-E3, IC23 DG468DV-T1-E3, IC24 DG468DV-T1-E3, IC25 DG468DV-T1-E3, IC26 DG468DV-T1-E3, IC27 DG468DV-T1-E3, IC28 DG468DV-T1-E3, IC29 DG468DV-T1-E3, IC3 Si8641BB-B-IS1, IC30 DG468DV-T1-E3, IC31 DG468DV-T1-E3, IC32 DG468DV-T1-E3, IC33 DG468DV-T1-E3, IC34 DG468DV-T1-E3, IC35 OPA376AIDBVR, IC36 ADS8674IDBT, IC4 L78L12, IC5 LM1117MP-5.0, IC6 LP2985-33DBVR, IC7 L79L12, IC8 STM32F446ZCT6, IC9 OPA2196IDR, J1 4907, J2 N.C., Q1 2N7002PS,115, Q10 BSS169, Q11 BSS169, Q12 BSS169, Q13 BSS169, Q2 2N7002PS,115, Q3 2N7002PS,115, Q4 2N7002PS,115, Q5 2N7002PS,115, Q6 BSS169, Q7 BSS169, Q8 BSS169, Q9 BSS169, X1 77317-104-28LF, X2 SSW-106-02-S-S, X3 691327310016, X4 691327310016, X5 1-2314878-0, X6 1-2314878-0, X7 1-2314878-0, Y1 25MHz

Commit message: r2B4 version
Parts:
- removed C89: 4n7/1kV, rcl:C-EUC1812
- removed C90, C91, C97, C98: 1n, rcl:C-EUC0805
- removed C92, C95, C96: 10u, rcl:C-EUC1206
- removed C93: 1u, rcl:C-EUC0805
- removed C94: 22u, rcl:C-EUC1206
- removed IC23, IC24, IC25, IC26, IC27, IC28, IC29, IC30, IC31, IC32, IC33, IC34: DG468DV-T1-E3, EEZ_DIB:DG468DV-T1-E3
- removed IC35: OPA376AIDBVR, EEZ_TI:OPA376AIDBVR
- removed IC36: ADS8674IDBT, EEZ_TI:ADS8674IDBT
- removed JP10, JP12, JP8: DS1025-01-1*2P8BV1-B, EEZ_Lib1:JUMPER-2PIN-2MM
- removed JP11, JP9: JP2-CUT-0805, EEZ_Lib1:JP2-CUT-0805
- removed L10, L11, L12, L8, L9: BLM18AG102SH1D, EEZ_Lib1:FERRITE_BEAD0603
- removed Q12, Q13: BSS169, EEZ_Lib1:BSS169
- removed R66, R72, R76, R80: 47R, rcl:R-EU_R0805
- removed R67, R70, R73, R74, R77, R78, R81, R82: 100R, rcl:R-EU_R0805
- removed R68, R69: N.C., rcl:R-EU_R0805
- removed R71, R75, R79, R83: 154R, rcl:R-EU_R0805
- removed TR2: MDD02M-15, EEZ_inductors_and_transformers:MDD02
- removed TVS5, TVS6, TVS7, TVS8: PESD12VL1BA,115, EEZ_Lib1:PESDXL1BA
- added C22: 4n7/1kV, rcl:C-EUC1812
- added D15, D16, D17, D18, D19, D20, D21, D22, D27, D28: BAT54SFILM, diode:BAT54S
- added D23, D24, D25, D26: BAS316, EEZ_Lib1:DIODESOD323R
- added D29, D30: MBR0530T3G, EEZ_Lib1:SCHOTTKYSOD123
- added K1, K2: TQ2SS-L2-5V-X, EEZ_switches:TQ2SS-L2RELAY_TQ2_SS_PAN-M
- added RN6: DR1206-33R-4/8, EEZ_Lib1:R_ARRAY4
- added X8: DS1023-2*14S21, EEZ_connectors:TSW-114-07-F-D
- added ZD3: SMAJ16A, EEZ_Lib1:SMAJ-ADO214AC
- C10: value 100n -> 1u; device rcl:C-EUC0603 -> rcl:C-EUC0805
- C12: value 4n7/1kV -> 4u7; device rcl:C-EUC1812 -> rcl:C-EUC0805
- C14: value 2u2 -> 1u
- C15, C8: value 1u -> 4u7
- C16, C47, C57, C58: value 4u7 -> 100n; device rcl:C-EUC0805 -> rcl:C-EUC0603
- C17: value 10n -> 1u
- C18, C35, C72, C73, C87, C88: value 1u -> 100n; device rcl:C-EUC0805 -> rcl:C-EUC0603
- C19: value N.C. -> 1u
- C20: value 18p -> 10u; device rcl:C-EUC0603 -> rcl:C-EUC1206
- C21: value 18p -> 1u; device rcl:C-EUC0603 -> rcl:C-EUC0805
- C23: device EEZ_Lib1:ECAP1206 -> rcl:C-EUC0805
- C24: value 100n -> N.C.; device rcl:C-EUC0603 -> rcl:C-EUC0805
- C25, C26: value 100n -> 4p7
- C27: value 100n -> 4u7; device rcl:C-EUC0603 -> EEZ_Lib1:ECAP1206
- C37, C38: value 2u2 -> 100n; device rcl:C-EUC0805 -> rcl:C-EUC0603
- C39: value 2n2 -> 1u
- C40, C49, C60, C66: value 1n -> 100n; device rcl:C-EUC0805 -> rcl:C-EUC0603
- C41: value 100n -> 2u2; device rcl:C-EUC0603 -> rcl:C-EUC0805
- C42: value 22n -> 2u2
- C43, C52: value 100n -> 2n2; device rcl:C-EUC0603 -> rcl:C-EUC0805
- C44, C53, C70: value 100n -> 1n; device rcl:C-EUC0603 -> rcl:C-EUC0805
- C46: value 4u7 -> 22n
- C48: value 2n2 -> 100n; device rcl:C-EUC0805 -> rcl:C-EUC0603
- C50, C62, C68: value 100n -> 4u7; device rcl:C-EUC0603 -> rcl:C-EUC0805
- C51: value 22n -> 4u7
- C55: value 100n -> 22n; device rcl:C-EUC0603 -> rcl:C-EUC0805
- C6: value 4n7/1kV -> 100n; device rcl:C-EUC1812 -> rcl:C-EUC0603
- C61: value 150n -> 4u7
- C64: value 4u7 -> 1n
- C65: value 100n -> 150n; device rcl:C-EUC0603 -> rcl:C-EUC0805
- C7: value 1u -> 2u2
- C75: value 10u -> 100n; device rcl:C-EUC1206 -> rcl:C-EUC0603
- C76: value 330p -> 10u; device rcl:C-EUC0805 -> rcl:C-EUC1206
- C77: value 330p -> 100p
- C78, C86: value 100n -> 100p; device rcl:C-EUC0603 -> rcl:C-EUC0805
- C79, C80, C81, C82, C83, C84, C85: value 100n -> 10n; device rcl:C-EUC0603 -> rcl:C-EUC0805
- C9: value 1u -> 10n
- D1, D10, D2, D3, D4, D5, D6, D7, D8, D9: value BAT54SFILM -> MBR0530T3G; device diode:BAT54S -> EEZ_Lib1:SCHOTTKYSOD123
- D11, D12, D13, D14: value BAT54SFILM -> N.C.
- IC10: value DAC7760IPWPR -> OPA2196IDR; device EEZ_TI:DAC7760IPWPR -> EEZ_Lib1:TL072SOIC8
- IC12: value OPA376AIDBVR -> DAC7760IPWPR; device EEZ_TI:OPA376AIDBVR -> EEZ_TI:DAC7760IPWPR
- IC13: value DAC7563TDGSR -> OPA376AIDBVR; device EEZ_TI:DAC7563TDGSR -> EEZ_TI:OPA376AIDBVR
- IC14: value OPA2196IDR -> DAC7563TDGSR; device EEZ_Lib1:TL072SOIC8 -> EEZ_TI:DAC7563TDGSR
- IC15: value BTS3408G -> OPA2196IDR; device EEZ_Lib1:BTS3408G -> EEZ_Lib1:TL072SOIC8
- IC19: value 74HC126PW,118 -> BTS3408G; device EEZ_DIB:74HC126PW,118 -> EEZ_Lib1:BTS3408G
- IC21, IC22: value DG468DV-T1-E3 -> 74HC126PW,118; device EEZ_DIB:DG468DV-T1-E3 -> EEZ_DIB:74HC126PW,118
- IC4: value L78L12 -> LP2985-33DBVR; device EEZ_Lib1:MC78LXXSOIC8 -> EEZ_DIB:LP2985
- IC5: value LM1117MP-5.0 -> L78L15; device EEZ_Lib1:LM1117MP-5.0 -> EEZ_Lib1:MC78LXXSOIC8
- IC6: value LP2985-33DBVR -> SN6505BDBVT; device EEZ_DIB:LP2985 -> EEZ_TI:SN6505BDBVT
- IC7: value L79L12 -> L79L15
- IC9: value OPA2196IDR -> (none); device EEZ_Lib1:TL072SOIC8 -> EEZ_DIB:XTSD0XG
- JP2, JP3: value JP2-CUT-0805 -> DS1025-01-1*3P8BV1-B; device EEZ_Lib1:JP2-CUT-0805 -> EEZ_connectors:JUMPER-3PIN2MM
- JP6: value JP3-CUT-0805-ROTATED -> DS1025-01-1*3P8BV1-B; device EEZ_Lib1:JP3-CUT-0805-ROTATED -> EEZ_connectors:JUMPER-3PIN2MM
- JP7: value DS1025-01-1*2P8BV1-B -> DS1025-01-1*3P8BV1-B; device EEZ_Lib1:JUMPER-2PIN-2MM -> EEZ_connectors:JUMPER-3PIN2MM
- L1: value DLW21SN371SQ2L -> SRF0905-202Y; device EEZ_inductors_and_transformers:DLW21S -> EEZ_inductors_and_transformers:SRF0905
- L2, L3: value DLW21SN371SQ2L -> BLM18AG102SH1D; device EEZ_inductors_and_transformers:DLW21S -> EEZ_Lib1:FERRITE_BEAD0603
- Q10, Q9: value BSS169 -> MMBT5551; device EEZ_Lib1:BSS169 -> transistor:MMBT5551LT1-NPN-SOT23-BEC
- Q11: value BSS169 -> 2N7002; device EEZ_Lib1:BSS169 -> EEZ_Lib1:2N7002
- Q6, Q8: value BSS169 -> BSS84P; device EEZ_Lib1:BSS169 -> EEZ_Lib1:IRLML2246TRPBF
- Q7: value BSS169 -> MMBT5401; device EEZ_Lib1:BSS169 -> transistor:BC857B-PNP-SOT23-BEC
- R1, R2: value N.C. -> 470K
- R10, R5: value N.C. -> 10K
- R12: value 10K -> N.C.
- R14: value N.C. -> 9K09 0.1%
- R15: value 15R -> 75K 0.1%
- R17: value 75K 0.1% -> 180R
- R18: value 9K09 0.1% -> 47R
- R19, R26: value 180R -> 9K09 0.1%
- R20: value 47R -> 9K09 0.1%
- R21: value 9K09 0.1% -> 75K 0.1%
- R24: value 9K09 0.1% -> 180R
- R25: value 75K 0.1% -> 47R
- R27: value 47R -> 75K 0.1%
- R28: value 9K09 0.1% -> 10K
- R29: value 75K 0.1% -> 100R
- R30, R62: value 10K -> 470R
- R31: value 100R -> 1K8
- R32, R33: value 100R -> 2K7; device rcl:R-EU_R0805 -> rcl:R-EU_R1206
- R34: value 470R -> 2K7; device rcl:R-EU_R0805 -> rcl:R-EU_R1206
- R35: value 1K8 -> 2K7; device rcl:R-EU_R0805 -> rcl:R-EU_R1206
- R4: value N.C. -> 4K7
- R40, R41, R42, R43: value 2K7 -> 27K; device rcl:R-EU_R1206 -> rcl:R-EU_R0805
- R48, R49, R50, R51: value 27K -> 1K
- R56: value 1K -> 100K
- R57, R58: value 1K -> 100R
- R59: value 1K -> 47R
- R6: value 4K7 -> 47R
- R60: value 470K -> 100K; device rcl:R-EU_R1206 -> rcl:R-EU_R0805
- R61: value 470K -> 10K; device rcl:R-EU_R1206 -> rcl:R-EU_R0805
- R64: value N.C. -> 100K
- R65: value N.C. -> 47R
- R7: value 10K -> 15R
- R8: value 47R -> N.C.
- RN3: value DR1206-10K-4/8 -> DR1206-47K-4/8
- RN4: value DR1206-33R-4/8 -> N.C.
- TR1: value TBA2-1223 -> WE-750315371; device EEZ_inductors_and_transformers:TBA-DUAL-2W -> EEZ_inductors_and_transformers:MURATA_78615
- X2: value SSW-106-02-S-S -> N.C.
- X4: value 691327310016 -> 691322310008; device EEZ_connectors:691327310016 -> EEZ_connectors:691322310008
- X5, X6: value 1-2314878-0 -> DS1014-10RF1B; device EEZ_connectors:1-2314878-0 -> EEZ_connectors:DS1014-10RF1B
- X7: value 1-2314878-0 -> DS1023-2*14S21; device EEZ_connectors:1-2314878-0 -> EEZ_connectors:TSW-114-07-F-D
- Y1: value 25MHz -> LF XTAL026392; device EEZ_Lib1:XTALSMD -> EEZ_Lib1:12SMX-B
- ZD1: value MMSZ4700T1G -> MM3Z18VT1G; device EEZ_Lib1:ZENER-DIODESOD123 -> EEZ_Lib1:ZENER-DIODESOD323R
- ZD2: value MMSZ4700T1G -> SMAJ16A; device EEZ_Lib1:ZENER-DIODESOD123 -> EEZ_Lib1:SMAJ-ADO214AC
Connections:
- removed net !OUT_FAULT: IC15.!FAULT, IC16.!FAULT, IC17.!FAULT, IC18.!FAULT, IC8B.PG3, R30.2
- removed net +12V: C7.2, L1.4, X1-21.1, X1-22.1
- removed net +12V_CM: C6.1, C8.2, L1.3, TR1.IN+, TR2.IN+
- removed net +12V_ISO: C10.1, C45.1, C47.2, C53.1, C55.1, C58.2, C59.1, C67.2, C68.2, C69.2, C70.2, C72.1, D1.C2, D2.C2, D3.C2, D4.C2, IC10.AVDD, IC11.AVDD, IC14P.V+, IC15.VSS, IC16.VSS, IC17.VSS, IC18.VSS, IC4.VO, IC5.IN, IC9P.V+, JP2.2, JP4.3, ZD1.C
- removed net -12V_ISO: C13.2, C44.1, C46.2, C54.1, C56.1, C57.2, C62.1, C73.1, D1.A1, D2.A1, D3.A1, D4.A1, IC10.AVSS, IC10.EPAD, IC11.AVSS, IC11.EPAD, IC14P.V-, IC7.OUT, IC9P.V-, JP3.2, JP5.3, R64.1, R65.1, R68.1, R69.1, ZD2.C
- removed net ADC_AVDD: C86.1, C95.2, IC35P.V+, IC36.AVDD, L11.2, X5-3.1
- removed net ADC_IRQ: IC36.ALARM, IC8A.PD8, X5-9.1
- removed net ADC_SCLK: IC36.SCLK, RN5-2.1, X5-7.1
- removed net ADC_VREF: C92.2, IC35A.+IN, IC36.REFIO, X7-2.1
- removed net AGND2: JP8.1, R74.1, R75.1, TVS6.1, X4-4.1, X6-6.1
- removed net AGND4: JP12.1, R82.1, R83.1, TVS8.1, X4-8.1, X610.1
- removed net AIN0: L8.2, Q6.D, R62.2, TVS5.2
- removed net AIN1: L9.2, Q8.D, R63.2, TVS6.2
- removed net AIN_0GND: C90.1, IC36.AIN_0GND, R71.2, X7-4.1
- removed net AIN_0P: C90.2, IC36.AIN_0P, R64.2, R67.2, X7-3.1
- removed net AIN_1GND: C91.1, IC36.AIN_1GND, R75.2, X7-6.1
- removed net AIN_1P: C91.2, IC36.AIN_1P, R65.2, R73.2, X7-5.1
- removed net AIN_2GND: C97.1, IC36.AIN_2GND, R79.2, X7-8.1
- removed net AIN_2P: C97.2, IC36.AIN_2P, R68.2, R77.2, X7-7.1
- removed net AIN_3GND: C98.1, IC36.AIN_3GND, R83.2, X710.1
- removed net AIN_3P: C98.2, IC36.AIN_3P, R69.2, R81.2, X7-9.1
- removed net CURR_SW0: IC22A.IN, IC27A.IN, IC8A.PD3
- removed net CURR_SW1: IC23A.IN, IC28A.IN, IC8A.PD4
- removed net CURR_SW2: IC24A.IN, IC29A.IN, IC8A.PD5
- removed net CURR_SW3: IC25A.IN, IC30A.IN, IC8A.PD6
- removed net DAC_SCLK: IC10.SCLK, IC11.SCLK, IC13.SCLK, RN4-2.1
- removed net DIN7: C85.1, D14.C1A2, IC8A.PB7, R43.2, R51.2, R59.1
- removed net GND_CM: C12.1, C8.1, L1.2, TR1.IN-, TR2.IN-
- removed net N$103: IC8A.PA7, RN4-4.2
- removed net N$126: IC21B.NO, R62.1
- removed net N$130: IC26B.NO, R63.1
- removed net N$136: JP9.1, L10.2, Q10.D, TVS7.2
- removed net N$137: JP11.1, L12.2, Q12.D, TVS8.2
- removed net N$2: Q12.G, Q13.S, R80.1
- removed net N$30: IC30B.NO, IC34B.NO, Q13.D
- removed net N$31: IC35A.-IN, IC35A.OUT, JP6.NC
- removed net N$32: Q8.G, Q9.S, R72.1
- removed net N$35: C93.2, C94.2, IC36.REFCAP
- removed net N$37: IC8A.PB13, RN5-2.2
- removed net N$47: C9.2, L2.1, TR1.OUT+, TR2.OUT+
- removed net N$48: C12.2, C18.2, C6.2, C9.1, L2.4, L3.1, TR1.COMM, TR2.COMM
- removed net N$49: C18.1, L3.4, TR1.OUT-, TR2.OUT-
- removed net N$50: IC23B.NO, IC28B.COM, R74.2
- removed net N$51: IC23B.COM, IC32B.COM, R73.1
- removed net N$75: IC28B.NO, IC32B.NO, Q9.D
- removed net N$77: Q10.G, Q11.S, R76.1
- removed net N$78: Q6.G, Q7.S, R66.1
- removed net N$81: IC8A.PA4, RN4-1.2
- removed net N$84: Q10.S, Q11.G, R76.2
- removed net N$85: IC24B.NO, IC29B.COM, R78.2
- removed net N$86: Q6.S, Q7.G, R66.2
- removed net N$87: IC24B.COM, IC33B.COM, JP9.2, R77.1
- removed net N$88: IC29B.NO, IC33B.NO, Q11.D
- removed net N$89: IC22B.NO, IC27B.COM, R70.2
- removed net N$91: L8.1, X4-1.1, X6-1.1
- removed net N$92: IC22B.COM, IC31B.COM, R67.1
- removed net N$93: L9.1, X4-3.1, X6-5.1
- removed net N$94: L10.1, X4-5.1, X6-7.1
- removed net N$95: IC27B.NO, IC31B.NO, Q7.D
- removed net N$96: L12.1, X4-7.1, X6-9.1
- removed net N$98: IC8A.PA5, RN4-2.2
- removed net OUT_EN: IC15.ENA, IC16.ENA, IC17.ENA, IC18.ENA, IC19A.EN, IC19B.EN, IC19C.EN, IC19D.EN, IC8A.PB11
- removed net PWM#1: IC19A.I, IC19B.I, IC8A.PD12
- removed net PWM#2: IC19C.I, IC19D.I, IC8A.PA3
- removed net SCLK: IC8B.PE12, RN1-2.2
- removed net TEMP_SW#1: IC21A.IN, IC8A.PC13
- removed net TEMP_SW#2: IC26A.IN, IC8A.PC14-OSC32_IN
- removed net VOLT_SW0: IC31A.IN, IC8B.PF0
- removed net VOLT_SW1: IC32A.IN, IC8B.PF1
- removed net VOLT_SW2: IC33A.IN, IC8B.PF2
- removed net VOLT_SW3: IC34A.IN, IC8B.PF3
- new net !ADC_DRDY: IC8B.PG15, X7-7.1
- new net !DOUT_FAULT: IC16.!FAULT, IC17.!FAULT, IC18.!FAULT, IC19.!FAULT, IC8B.PG1, R28.2
- new net +5V: L1.1, X1-23.1, X1-24.1
- new net -15V_IN: C17.1, IC7.IN, L3.2
- new net -5V_ISO: C23.2, D10.A, D9.A, X7-15.1
- new net ADC_CLK/SCL1: IC8A.PB7, X7-4.1
- new net ADC_SCK: RN5-2.1, X7-6.1
- new net ADC_START/SDA1: IC8A.PB6, X7-10.1
- new net ADIB1N: JP2.2, K1G$2.NC, X5-3.1
- new net ADIB1P: JP3.2, K1G$3.NC, X5-4.1
- new net ADIB1_ID0: IC8A.PD13, X5-7.1
- new net ADIB1_ID1: IC8A.PD12, X5-9.1
- new net ADIB1_ID2: IC8A.PD11, X5-8.1
- new net ADIB1_R: IC21B.I, IC8A.PA9
- new net ADIB1_S: IC21A.I, IC8A.PD3
- new net ADIB2N: JP4.2, K2G$2.NC, X6-3.1
- new net ADIB2P: JP5.2, K2G$3.NC, X6-4.1
- new net ADIB2_ID0: IC8B.PG2, X6-7.1
- new net ADIB2_ID1: IC8A.PD15, X6-9.1
- new net ADIB2_ID2: IC8A.PD14, X6-8.1
- new net ADIB2_R: IC21D.I, IC8A.PA11
- new net ADIB2_S: IC21C.I, IC8A.PA10
- new net AFE1N: JP2.1, K1G$2.COM, X7-25.1
- new net AFE1P: JP3.3, K1G$3.COM, X7-26.1
- new net AFE2N: JP4.3, K2G$2.COM, X7-23.1
- new net AFE2P: JP5.1, K2G$3.COM, X7-24.1
- new net AFE_CLK: IC8A.PA8, X7-14.1
- new net AFE_ID0: IC8B.PE9, X8-1.1
- new net AFE_ID1: IC8B.PE8, X8-2.1
- new net BIAS_EN: IC8B.PE7, R62.1
- new net DAC_SCK: IC11.SCLK, IC12.SCLK, IC14.SCLK, RN6-2.1
- new net DIN7/MISO: C86.1, D22.C1A2, IC8A.PA6, R39.2, R47.2, R55.1
- new net DOUT_EN: IC16.ENA, IC17.ENA, IC18.ENA, IC19.ENA, IC22A.EN, IC22B.EN, IC22C.EN, IC22D.EN, IC8A.PA4
- new net ISEL#1: IC8B.PG14, X8-3.1
- new net ISEL#2: IC8A.PC15-OSC32_OUT, X8-4.1
- new net ISEL10_R#3: IC8A.PD6, X8-21.1
- new net ISEL10_R#4: IC8A.PC1, X8-22.1
- new net ISEL10_S#3: IC8A.PD7, X8-19.1
- new net ISEL10_S#4: IC8B.PF5, X8-20.1
- new net ISEL_LOW#3: IC8A.PD5, X8-23.1
- new net ISEL_LOW#4: IC8A.PC2, X8-24.1
- new net ISEL_MID#3: IC8A.PD4, X8-25.1
- new net ISEL_MID#4: IC8A.PC3, X8-26.1
- new net ISEL_R#3: IC8B.PG9, X8-17.1
- new net ISEL_R#4: IC8B.PF4, X8-18.1
- new net ISEL_S#3: IC8B.PG10, X8-15.1
- new net ISEL_S#4: IC8B.PF3, X8-16.1
- new net N$104: C19.1, D6.A, D7.C
- new net N$105: C21.1, D7.A, D8.C
- new net N$111: C14.2, IC5.VI, L2.2
- new net N$149: Q8.G, Q9.C, R61.2
- new net N$151: Q6.G, Q7.C, R60.2, R61.1
- new net N$152: D29.A, Q6.D
- new net N$153: D29.C, JP6.3, ZD2.C
- new net N$154: Q6.S, Q7.B, R59.2, R60.1
- new net N$155: Q10.C, Q11.G, R63.2, R64.1
- new net N$162: Q10.B, Q11.S, R64.2, R65.2
- new net N$163: Q8.D, R63.1
- new net N$164: D30.C, Q11.D
- new net N$167: C15.2, D8.A, L3.1
- new net N$168: D30.A, JP7.3, ZD3.A
- new net N$169: C12.1, D3.C, L2.1
- new net N$176: IC8A.PB12, RN6-1.2
- new net N$177: IC8A.PB13, RN6-2.2
- new net N$178: IC8A.PB14, RN6-3.2
- new net N$179: IC8A.PB15, RN6-4.2
- new net N$52: C11.1, D4.A, D5.C
- new net N$53: IC6.D2, TR1.1
- new net N$63: IC6.D1, TR1.3
- new net N$64: C11.2, C19.2, D1.A, D9.C, TR1.6
- new net N$70: C10.2, C21.2, D10.C, D2.A, TR1.4
- new net N$79: C10.1, D3.A, D4.C
- new net PWM#1/SCK: IC22A.I, IC22B.I, IC8A.PA5
- new net PWM#2/MOSI: IC22C.I, IC22D.I, IC8A.PA7
- new net SCK: IC8B.PE12, RN2-2.2
- new net SN_GND: C18.2, C20.1, IC6.CLK, IC6.GND, L1.3
- new net SN_VCC: C18.1, C20.2, IC6.EN, IC6.VCC, L1.4, TR1.2
- new net USEL1#1: IC8B.PG13, X8-5.1
- new net USEL1#2/SDA2: IC8B.PF0, X8-6.1
- new net USEL1#3: IC8A.PD1, X8-11.1
- new net USEL1#4: IC8A.PC13, X8-12.1
- new net USEL10#1: IC8B.PG12, X8-7.1
- new net USEL10#2/SCL2: IC8B.PF1, X8-8.1
- new net USEL10#3: IC8A.PD0, X8-13.1
- new net USEL10#4: IC8A.PC14-OSC32_IN, X8-14.1
- new net USEL100#1: IC8B.PG11, X8-9.1
- new net USEL100#2: IC8B.PF2, X8-10.1
- net !ADC_CS: now also X7-5.1; no longer IC36.!CS, X5-6.1
- net !DAC_ALARM: now also IC12.!ALARM, IC8A.PD8, R10.2; no longer IC10.!ALARM, IC8A.PC15-OSC32_OUT, R12.2
- net !DAC_CS_DUAL: now also IC14.!SYNC, RN6-1.1; no longer IC13.!SYNC, RN4-1.1
- net !RESET: now also IC14.!CLR, R4.2, X7-9.1; no longer IC13.!CLR, IC36.!RST/!PD, R6.2, X5-4.1
- net +15V_ISO: now also C13.1, C49.1, C51.2, C57.1, C59.1, C62.2, C63.1, C71.2, C72.2, C73.2, C74.2, D11.C2, D12.C2, D13.C2, D14.C2, IC10P.V+, IC11.AVDD, IC12.AVDD, IC15P.V+, IC16.VSS, IC17.VSS, IC18.VSS, IC19.VSS, IC5.VO, Q7.E, R59.1, X7-20.1; no longer C11.2, C87.1, IC21A.V+, IC22A.V+, IC23A.V+, IC24A.V+, IC25A.V+, IC26A.V+, IC27A.V+, IC28A.V+, IC29A.V+, IC30A.V+, IC31A.V+, IC32A.V+, IC33A.V+, IC34A.V+, IC4.VI, JP2.1, L2.2
- net +3V3_ISO: now also C27.+, C35.1, C36.1, C37.1, C38.1, C45.1, C54.1, C7.1, C88.2, IC12.DVDD, IC22P.V+, IC4.OUT, IC9.VDD, Q8.S, R10.1, R28.1, R29.1, RN4-1.1, RN4-2.1, RN4-3.1, RN4-4.1, X7-13.1; no longer C14.1, C19.1, C23.+, C25.1, C26.1, C27.1, C41.1, C50.1, C71.2, C96.2, D5.C2, D6.C2, IC10.DVDD, IC19P.V+, IC36.DVDD, IC6.OUT, R1.1, R12.1, R2.1, R30.1, R33.1, R5.1, R6.1, X510.1
- net +5V_ISO: now also C6.1, C8.2, C87.2, D1.C, D2.C, IC21P.V+, IC4.IN, IC4.ON/!OFF, K1G$1.R+, K1G$1.S+, K2G$1.R+, K2G$1.S+, R56.1, X7-16.1, ZD1.A; no longer C16.2, IC5.OUT, IC5.VOUT, IC6.IN, IC6.ON/!OFF, L11.1, X5-2.1
- net +VSENSE1: now also IC10A.-IN, IC10A.OUT, IC11.+VSENSE; no longer IC10.+VSENSE, IC9A.-IN, IC9A.OUT
- net +VSENSE2: now also IC10B.-IN, IC10B.OUT, IC12.+VSENSE; no longer IC11.+VSENSE, IC9B.-IN, IC9B.OUT
- net -15V_ISO: now also C16.2, C48.1, C50.2, C58.1, C60.1, C61.2, C66.1, D11.A1, D12.A1, D13.A1, D14.A1, IC10P.V-, IC11.AVSS, IC11.EPAD, IC12.AVSS, IC12.EPAD, IC15P.V-, IC7.OUT, Q10.E, R65.1, X7-19.1; no longer C15.1, C88.1, IC21A.V-, IC22A.V-, IC23A.V-, IC24A.V-, IC25A.V-, IC26A.V-, IC27A.V-, IC28A.V-, IC29A.V-, IC30A.V-, IC31A.V-, IC32A.V-, IC33A.V-, IC34A.V-, IC7.IN, JP3.1, L3.3
- net -VSENSE: now also IC12.-VSENSE, JP2.3, JP4.1, K1G$2.NO, K2G$2.NO; no longer IC10.-VSENSE
- net 1V25_REF: now also IC13A.-IN, IC13A.OUT, R14.2, R22.2; no longer IC12A.-IN, IC12A.OUT, JP6.NO, R16.2, R24.2
- net 2V5_REF: now also C65.2, IC14.VREF, R16.1; no longer C61.2, IC13.VREF, R18.1
- net ADC_MISO: now also X7-8.1; no longer IC36.SDO, X5-8.1
- net ADC_MOSI: now also X7-3.1; no longer IC36.SDI, X5-5.1
- net BOOT0: now also R5.2; no longer R7.2
- net CLAMP: now also C76.1, D15.C2, D16.C2, D17.C2, D18.C2, D19.C2, D20.C2, D21.C2, D22.C2, D27.C2, D28.C2, R29.2, R30.1; no longer C74.1, D10.C2, D11.C2, D12.C2, D13.C2, D14.C2, D7.C2, D8.C2, D9.C2, R33.2, R34.1
- net DAC_CLR#1: now also IC11.CLR, IC8B.PF12; no longer IC10.CLR, IC8B.PF9
- net DAC_CLR#2: now also IC12.CLR, IC8B.PF15; no longer IC11.CLR, IC8B.PF7
- net DAC_CLR-SEL#1: now also IC11.CLR-SEL, IC8B.PF13; no longer IC10.CLR-SEL, IC8B.PF10
- net DAC_CLR-SEL#2: now also IC12.CLR-SEL, IC8B.PG0; no longer IC11.CLR-SEL, IC8B.PF8
- net DAC_CS#1: now also IC11.LATCH, IC8B.PF11; no longer IC10.LATCH, IC8A.PC1
- net DAC_CS#2: now also IC12.LATCH, IC8B.PF14; no longer IC11.LATCH, IC8B.PF6
- net DAC_MISO: now also IC12.SDO, RN6-3.1; no longer IC10.SDO, RN4-3.1
- net DAC_MOSI: now also IC12.DIN, IC14.DIN, RN6-4.1; no longer IC10.DIN, IC13.DIN, RN4-4.1
- net DAC_OUT#1: now also C44.1, D11.C1A2, JP3.1, K1G$3.NO; no longer C40.1, D1.C1A2
- net DAC_OUT#2: now also C53.1, D12.C1A2, JP5.3, K2G$3.NO; no longer C49.1, D2.C1A2
- net DIB_CSA: now also RN1-2.1; no longer RN2-2.1
- net DIB_MISO: now also RN1-1.1; no longer RN2-1.1
- net DIB_MOSI: now also RN1-4.1; no longer RN2-4.1
- net DIB_SCLK: now also RN1-3.1; no longer RN2-3.1
- net DIN0: now also C77.1, C82.1, D15.C1A2, IC8B.PE6, R32.2, R40.2, R48.1; no longer C76.1, C81.1, D7.C1A2, IC8A.PA0-WKUP, R36.2, R44.2, R52.1
- net DIN1: now also C78.1, C83.1, D16.C1A2, IC8B.PE5, R33.2, R41.2, R49.1; no longer C77.1, C82.1, D8.C1A2, IC8A.PA1, R37.2, R45.2, R53.1
- net DIN2: now also C79.1, D17.C1A2, IC8B.PE4, R34.2, R42.2, R50.1; no longer C78.1, D9.C1A2, IC8A.PC6, R38.2, R46.2, R54.1
- net DIN3: now also C84.1, D18.C1A2, IC8B.PE3, R35.2, R43.2, R51.1; no longer C83.1, D10.C1A2, IC8A.PC7, R39.2, R47.2, R55.1
- net DIN4: now also C80.1, D19.C1A2, IC8B.PE2, R36.2, R44.2, R52.1; no longer C79.1, D11.C1A2, IC8A.PB4, R40.2, R48.2, R56.1
- net DIN5: now also C85.1, D20.C1A2, IC8B.PE1, R37.2, R45.2, R53.1; no longer C84.1, D12.C1A2, IC8A.PB5, R41.2, R49.2, R57.1
- net DIN6: now also C81.1, D21.C1A2, IC8B.PE0, R38.2, R46.2, R54.1; no longer C80.1, D13.C1A2, IC8A.PB6, R42.2, R50.2, R58.1
- net DOUT0: now also IC19.IN2, IC8A.PA0-WKUP; no longer IC18.IN1, IC8A.PA2
- net DOUT1: now also IC19.IN1, IC8A.PA1; no longer IC18.IN2, IC8A.PA9
- net DOUT2: now also IC18.IN2, IC8A.PA2; no longer IC17.IN1, IC8B.PG6
- net DOUT3: now also IC18.IN1, IC8A.PA3; no longer IC17.IN2, IC8B.PG7
- net DOUT4: now also IC17.IN2; no longer IC16.IN1
- net DOUT5: now also IC17.IN1; no longer IC16.IN2
- net DOUT6: now also IC16.IN1; no longer IC15.IN1
- net DOUT7: now also IC16.IN2; no longer IC15.IN2
- net GND: now also C12.2, C13.2, C14.1, C15.1, C17.2, C22.2, C23.1, C25.1, C26.1, C27.-, C37.2, C38.2, C39.2, C41.1, C47.2, C48.2, C50.1, C55.1, C57.2, C58.2, C6.2, C62.1, C64.2, C65.1, C67.2, C69.2, C7.2, C70.2, C72.1, C73.1, C74.1, C8.1, C81.2, C87.1, C88.1, C9.1, D15.A1, D16.A1, D17.A1, D18.A1, D19.A1, D20.A1, D21.A1, D22.A1, D27.A1, D28.A1, D5.A, D6.C, IC12.DVDD-EN, IC12.GND, IC13P.V-, IC14.!LDAC, IC14.GND, IC21P.V-, IC22P.V-, IC5.GND, IC9.VSS, Q9.E, R12.1, R2.2, R20.2, R21.2, R27.2, R31.2, R40.1, R41.1, R42.1, R43.1, R5.1, R8.1, TR1.5, X5-10.1, X5-2.1, X5-5.1, X5-6.1, X6-1.1, X6-10.1, X6-2.1, X6-5.1, X6-6.1, X7-11.1, X7-12.1, X7-2.1, X7-21.1, X7-22.1, X7-27.1, X7-28.1, X8-27.1, X8-28.1, ZD3.C; no longer C10.2, C11.1, C13.1, C14.2, C15.2, C17.1, C19.2, C20.1, C21.1, C23.-, C25.2, C26.2, C27.2, C37.1, C38.1, C41.2, C43.2, C47.1, C50.2, C52.2, C55.2, C57.1, C58.1, C62.2, C64.1, C65.2, C67.1, C69.1, C70.1, C72.2, C73.2, C74.2, C83.2, C87.2, C88.2, C89.2, C92.1, C93.1, C94.1, C95.1, C96.1, D10.A1, D11.A1, D12.A1, D13.A1, D14.A1, D5.A1, D6.A1, D7.A1, D8.A1, D9.A1, IC10.DVDD-EN, IC10.GND, IC12P.V-, IC13.!LDAC, IC13.GND, IC19P.V-, IC21A.GND, IC22A.GND, IC23A.GND, IC24A.GND, IC25A.GND, IC26A.GND, IC27A.GND, IC28A.GND, IC29A.GND, IC30A.GND, IC31A.GND, IC32A.GND, IC33A.GND, IC34A.GND, IC35P.V-, IC36.!REFSEL, IC36.AGND, IC36.AUX_GND, IC36.DAISY, IC36.DGND, IC36.REFGND, IC5.ADJ/GND, IC6.GND, JP10.2, JP12.2, JP7.2, JP8.2, L2.3, L3.2, R10.1, R14.1, R22.2, R23.2, R29.2, R35.2, R48.1, R49.1, R50.1, R51.1, R61.2, R7.1, ZD1.A
- net GNDIO: now also L1.2; no longer C7.1, L1.1
- net HART#1: now also C46.2, IC11.HART-IN; no longer C42.2, IC10.HART-IN
- net HART#2: now also C55.2, IC12.HART-IN; no longer C51.2, IC11.HART-IN
- net IN_CTRL0: now also IC8A.PC7, Q1A.G; no longer IC8A.PD7, Q2A.G
- net IN_CTRL1: now also IC8A.PC6, Q1B.G; no longer IC8B.PG9, Q2B.G
- net IN_CTRL2: now also IC8B.PG8, Q2A.G; no longer IC8B.PG10, Q3A.G
- net IN_CTRL3: now also IC8B.PG7, Q2B.G; no longer IC8B.PG11, Q3B.G
- net IN_CTRL4: now also IC8B.PG6, Q3A.G; no longer IC8B.PG12, Q4A.G
- net IN_CTRL5: now also IC8B.PG5, Q3B.G; no longer IC8B.PG13, Q4B.G
- net IN_CTRL6: now also IC8B.PG4, Q4A.G; no longer IC8B.PG14, Q5A.G
- net IN_CTRL7: now also IC8B.PG3, Q4B.G; no longer IC8A.PB3, Q5B.G
- net ISET1: now also R17.2, R18.1; no longer R19.2, R20.1
- net ISET2: now also R24.2, R25.1; no longer R26.2, R27.1
- net MISO: now also RN2-3.2; no longer RN1-3.2
- net MOSI: now also RN2-4.2; no longer RN1-4.2
- net N$1: now also IC19.GND; no longer IC15.GND
- net N$10: now also Q2A.D, R50.2; no longer Q3A.D, R54.2
- net N$100: now also IC8A.PB5, RN5-4.2; no longer IC8A.PA6, RN4-3.2
- net N$101: now also RN1-1.2; no longer RN2-1.2
- net N$102: now also RN1-4.2; no longer RN2-4.2
- net N$106: now also C9.2, IC4.BYPASS; no longer C17.2, IC6.BYPASS
- net N$109: now also R36.1, X4-4.1; no longer R40.1, X4-13.1
- net N$113: now also C42.2; no longer C38.2
- net N$115: now also C39.1, C40.1, R6.1; no longer C35.1, C36.1, R8.1
- net N$116: now also RN2-2.1; no longer RN1-2.1
- net N$118: now also RN2-1.1; no longer RN1-1.1
- net N$119: now also R38.1, X4-2.1; no longer R42.1, X4-15.1
- net N$12: now also RN2-4.1; no longer RN1-4.1
- net N$120: now also R39.1, X4-1.1; no longer R43.1, X4-16.1
- net N$121: now also R6.2; no longer R8.2
- net N$122: now also R37.1, X4-3.1; no longer R41.1, X4-14.1
- net N$129: now also D27.C1A2, IC22A.O, IC22B.O, R57.2; no longer D5.C1A2, IC19A.O, IC19B.O, JP4.1
- net N$13: now also Q2B.D, R51.2; no longer Q3B.D, R55.2
- net N$134: now also D28.C1A2, IC22C.O, IC22D.O, R58.2; no longer D6.C1A2, IC19C.O, IC19D.O, JP5.1
- net N$14: now also R33.1, X4-7.1; no longer R37.1, X4-10.1
- net N$15: now also Q3A.D, R52.2; no longer Q4A.D, R56.2
- net N$16: now also Q3B.D, R53.2; no longer Q4B.D, R57.2
- net N$17: now also Q4A.D, R54.2; no longer Q5A.D, R58.2
- net N$19: now also C52.2, IC12.CMP; no longer C48.2, IC11.CMP
- net N$20: now also IC21A.EN, IC21B.EN, IC21C.EN, IC21D.EN, R56.2; no longer IC21B.COM, IC26B.COM, JP6.COM
- net N$21: now also R1.2, R2.1; no longer R60.2, R61.1
- net N$22: now also D23.A, IC21A.O, K1G$1.S-; no longer JP4.2, R31.1
- net N$23: now also Q4B.D, R55.2; no longer Q5B.D, R59.2
- net N$24: now also C82.2, Q5A.D; no longer C81.2, Q1A.D
- net N$25: now also JP6.2; no longer R31.2
- net N$26: now also C52.1, IC12.VOUT, R13.2; no longer C48.1, IC11.VOUT, R15.2
- net N$27: now also IC8A.PA15, RN5-1.2; no longer IC8A.PB14, RN5-3.2
- net N$28: now also D24.A, IC21B.O, K1G$1.R-; no longer IC25B.COM, IC34B.COM, JP11.2, R81.1
- net N$29: now also IC8A.PB3, RN5-2.2; no longer IC8A.PB15, RN5-4.2
- net N$3: now also Q9.B, R62.2; no longer JP10.1, R78.1, R79.1, TVS7.1, X4-6.1, X6-8.1
- net N$33: now also D23.C, D24.C, D25.C, D26.C, ZD1.C; no longer Q8.S, Q9.G, R72.2
- net N$34: now also IC8A.PB4, RN5-3.2; no longer IC8A.PB12, RN5-1.2
- net N$36: now also R32.1, X4-8.1; no longer R36.1, X4-9.1
- net N$38: now also R34.1, X4-6.1; no longer R38.1, X4-11.1
- net N$39: now also JP7.2; no longer R32.2
- net N$4: now also JP6.1, R57.1; no longer Q12.S, Q13.G, R80.2
- net N$40: now also D25.A, IC21C.O, K2G$1.S-; no longer JP5.2, R32.1
- net N$41: now also D26.A, IC21D.O, K2G$1.R-; no longer JP7.1, R70.1, R71.1, TVS5.1, X4-2.1, X6-2.1
- net N$42: now also R35.1, X4-5.1; no longer R39.1, X4-12.1
- net N$43: now also IC10B.+IN, R11.1; no longer IC9B.+IN, R15.1
- net N$45: now also IC12.IOUT, R11.2; no longer IC11.IOUT, R13.2
- net N$46: now also C56.1, IC12.REFIN, IC12.REFOUT; no longer C52.1, IC11.REFIN, IC11.REFOUT
- net N$54: now also IC15B.+IN, R19.1; no longer IC14B.+IN, R23.1
- net N$55: now also IC15B.-IN, R14.1, R15.2; no longer IC14B.-IN, R16.1, R17.2
- net N$56: now also IC15B.OUT, R17.1; no longer IC14B.OUT, R19.1
- net N$57: now also IC15A.+IN, R26.1, R27.1; no longer IC14A.+IN, R28.1, R29.1
- net N$58: now also IC15A.-IN, R22.1, R23.2; no longer IC14A.-IN, R24.1, R25.2
- net N$59: now also IC15A.OUT, R24.1; no longer IC14A.OUT, R26.1
- net N$6: now also JP7.1, R58.1; no longer IC25B.NO, IC30B.COM, R82.2
- net N$60: now also IC13A.+IN, R16.2, R20.1; no longer IC12A.+IN, R18.2, R22.1
- net N$61: now also IC14.VOUTA, R19.2; no longer IC13.VOUTA, R21.2
- net N$62: now also C43.2, IC11.CMP; no longer C39.2, IC10.CMP
- net N$65: now also IC10A.+IN, R7.1; no longer IC9A.+IN, R11.1
- net N$66: now also C47.1, IC11.REFIN, IC11.REFOUT; no longer C43.1, IC10.REFIN, IC10.REFOUT
- net N$67: now also IC14.VOUTB, R26.2; no longer IC13.VOUTB, R28.2
- net N$68: now also IC12.ISET-R, R12.2; no longer IC11.ISET-R, R14.2
- net N$69: now also RN1-2.2; no longer RN2-2.2
- net N$7: now also R30.2, R31.1; no longer R34.2, R35.1
- net N$71: now also C67.1, C68.2, C69.1, IC13P.V+, IC14.VDD; no longer C63.1, C64.2, C65.1, IC12P.V+, IC13.VDD
- net N$72: now also RN2-3.1; no longer RN1-3.1
- net N$73: now also C70.1, D14.C1A2, R23.1, R25.2; no longer C66.1, D4.C1A2, R25.1, R27.2
- net N$74: now also C64.1, D13.C1A2, R15.1, R18.2; no longer C60.1, D3.C1A2, R17.1, R20.2
- net N$76: now also C83.2, Q5B.D; no longer C82.2, Q1B.D
- net N$8: now also Q1A.D, R48.2; no longer Q2A.D, R52.2
- net N$80: now also IC11.ISET-R, R8.2; no longer IC10.ISET-R, R10.2
- net N$82: now also C43.1, IC11.VOUT, R9.2; no longer C39.1, IC10.VOUT, R11.2
- net N$83: now also IC11.IOUT, R7.2; no longer IC10.IOUT, R9.2
- net N$9: now also Q1B.D, R49.2; no longer Q2B.D, R53.2
- net N$97: now also C41.2; no longer C37.2
- net N$99: now also RN1-3.2; no longer RN2-3.2
- net NSS: now also RN2-1.2; no longer RN1-1.2
- net PE: now also C22.1, R1.1; no longer C89.1, R60.1
- net POUT0: now also IC19.OUT2; no longer IC18.OUT1
- net POUT1: now also IC19.OUT1; no longer IC18.OUT2
- net POUT2: now also IC18.OUT2; no longer IC17.OUT1
- net POUT3: now also IC18.OUT1; no longer IC17.OUT2
- net POUT4: now also IC17.OUT2; no longer IC16.OUT1
- net POUT5: now also IC17.OUT1; no longer IC16.OUT2
- net POUT6: now also IC16.OUT1; no longer IC15.OUT1
- net POUT7: now also IC16.OUT2; no longer IC15.OUT2
- net RCC_OSC_IN: now also C25.2; no longer C20.2
- net RCC_OSC_OUT: now also C26.2; no longer C21.2
- net SDIO_CLK: now also IC9.CLK
- net SDIO_CMD: now also IC9.CMD, RN4-2.2; no longer R4.2
- net SDIO_D0: now also IC9.DAT0, RN4-1.2; no longer R2.2
- net SDIO_D1: now also IC9.DAT1, R3.2; no longer R5.2
- net SDIO_D2: now also IC9.DAT2, RN4-4.2; no longer R3.2
- net SDIO_D3: now also IC9.CD/DAT3, RN4-3.2; no longer R1.2
- net SD_DETECT: now also IC8A.PA12; no longer IC8A.PA15
- net SLOW_DIN#0: now also IC8A.PB9, Q5A.G; no longer IC8A.PB8, Q1A.G
- net SLOW_DIN#1: now also IC8A.PB8, Q5B.G; no longer IC8A.PB9, Q1B.G
- net SYNC: now also IC8B.PE15; no longer IC8A.PD11
Other:
- note added: "!CS! 5"
- note added: "!DRDY! 7"
- note added: "!RESET! 9"
- note added: "+3V3 13"
- note added: "+5V3 15"
- note added: "-15V 19"
- note added: "10 PF2"
- note added: "10 SPI_MISO"
- note added: "12 Gnd"
- note added: "12 PC13"
- note added: "12-bit dual DAC with bipolar voltage outputs 8-ch digital low-side power outputs"
- note added: "14 AFE EXT CLK"
- note added: "14 PC14"
- note added: "16 -5V3"
- note added: "16 PF3"
- note added: "18 N.C."
- note added: "18 PF4"
- note added: "2 AFE_ID1"
- note added: "2 Gnd"
- note added: "20 +15V"
- note added: "20 PF5"
- note added: "22 Gnd"
- note added: "22 PC1"
- note added: "24 ADIB2P"
- note added: "24 PC2"
- note added: "26 ADIB1P"
- note added: "26 PC3"
- note added: "28 Gnd"
- note added: "28-pin AFE socket (lower)"
- note added: "28-pin AFE socket (upper)"
- note added: "4 ADC CLK SEL / I2C_SCL1"
- note added: "4 PC15"
- note added: "6 PF0 / I2C_SDA2"
- note added: "6 SPI_CLK"
- note added: "8 ADC_START / I2C_SDA1"
- note added: "8 PF1 / I2C_SCL2"
- note added: "ADC"
- note added: "ADIB signal switching"
- note added: "ADIB1N 25"
- note added: "ADIB2N 23"
- note added: "AFE connectors"
- note added: "AFE_ID0 1"
- note added: "AUX (shared with PWM#1, PWM#2, DIN7)"
- note added: "DACs"
- note added: "DACs with voltage/current bipolar outputs"
- note added: "DIB interface"
- note added: "Gnd 1"
- note added: "Gnd 21"
- note added: "Gnd 27"
- note added: "Isolated +/-5 V, +/-12 V power supply, +3.3 V LDO"
- note added: "Max. +10 mA"
- note added: "Max. -10 mA"
- note added: "N.C. 17"
- note added: "PD0 13"
- note added: "PD1 11"
- note added: "PD4 25"
- note added: "PD5 23"
- note added: "PD6 21"
- note added: "PD7 19"
- note added: "PG10 15"
- note added: "PG11 9"
- note added: "PG12 7"
- note added: "PG13 5"
- note added: "PG14 3"
- note added: "PG9 17"
- note added: "PWM outputs"
- note added: "PWM outputs / sensor bias ADIB and AFE connectors"
- note added: "SPI1"
- note added: "SPI2"
- note added: "SPI3"
- note added: "SPI4"
- note added: "SPI_MOSI 3"
- note added: "Sensor bias outputs"
- note removed: "+5V, +3V3 LDO"
- note removed: "12-bit DACs, voltage/current bipolar outputs"
- note removed: "12-bit dual DAC with voltage bipolar outputs 8-ch digital low-side power outputs, dual PWM"
- note removed: "ADC with switchable voltage/current inputs Temp sensors bias"
- note removed: "Analog input type selection (voltage/current)"
- note removed: "Bias for two temp. sensors"
- note removed: "C0G"
- note removed: "Isolated +/-12 V power supply"

Commit message: PCB ID added
Parts:
- IC9: value (none) -> N.C.
Connections:
- net GND: now also IC8A.PD10, IC8A.PD9
Other:
- note added: "PCB_ID0"
- note added: "PCB_ID0=0"
- note added: "PCB_ID1"
- moved on the sheet: C24, IC9, J2, R3, RN4-1, RN4-2, RN4-3, RN4-4
