File: EDA files/EEZ DIB MIO168 r2B5.brd (EAGLE design)
At the start: 146 x 95 mm, 266 parts, among them IC1 M24C32-WMN6P, IC10 OPA2196IDR, IC11 DAC7760IPWPR, IC12 DAC7760IPWPR, IC13 OPA376AIDBVR, IC14 DAC7563TDGSR, IC15 OPA2196IDR, IC16 BTS3408G, IC17 BTS3408G, IC18 BTS3408G, IC19 BTS3408G, IC2 Si8641BB-B-IS1, IC20 TL431B, IC21 74HC126PW,118, IC22 74HC126PW,118, IC3 Si8641BB-B-IS1, IC4 LP2985-33DBVR, IC5 L78L15, IC6 SN6505BDBVT, IC7 L79L15, IC8 STM32F446ZCT6, IC9 N.C., J1 4907, J2 N.C., K1 TQ2SS-L2-5V-X, K2 TQ2SS-L2-5V-X, Q1 2N7002PS,115, Q10 MMBT5551, Q11 2N7002, Q2 2N7002PS,115, Q3 2N7002PS,115, Q4 2N7002PS,115, Q5 2N7002PS,115, Q6 BSS84P, Q7 MMBT5401, Q8 BSS84P, Q9 MMBT5551, X1 77317-104-28LF, X2 N.C., X3 691327310016, X4 691322310008, X5 DS1014-10RF1B, X6 DS1014-10RF1B, X7 DS1023-2*14S21, X8 DS1023-2*14S21, Y1 LF XTAL026392

Commit message: r2B5, ADIB switcing
Parts:
- removed C88: 100n, rcl:C0603
- removed D27, D28: BAT54SFILM, diode:SOT23
- removed D29, D30: MBR0530T3G, EEZ_Lib1:SOD123
- removed JP4, JP5, JP6, JP7: DS1025-01-1*3P8BV1-B, EEZ_connectors:ZL303-03P
- removed K1, K2: TQ2SS-L2-5V-X, EEZ_switches:PANASONIC_TQ2_SS
- removed ZD3: SMAJ16A, EEZ_Lib1:DO214AC
- added R66: 47R, rcl:R0805
- C1: value 100n -> N.C.
- D23, D24: value BAS316 -> BAT54SFILM; device EEZ_Lib1:SOD323-R -> diode:SOT23
- D25, D26: value BAS316 -> MBR0530T3G; device EEZ_Lib1:SOD323-R -> EEZ_Lib1:SOD123
- IC21: value 74HC126PW,118 -> DG212BDY-T1-E3; device EEZ_DIB:PW14 -> EEZ_DIB:SO16
- R56: value 100K -> 1K
- R57: value 100R -> 1K
- R59: value 47R -> 100R
- R60: value 100K -> 47R
- R61: value 10K -> 100K
- R62: value 470R -> 10K
- R63: value 10K -> 470R
- R64: value 100K -> 10K
- R65: value 47R -> 100K
- ZD1: value MM3Z18VT1G -> SMAJ16A; device EEZ_Lib1:SOD323-R -> EEZ_Lib1:DO214AC
- moved JP2 68.7 mm to (23.4, 26.8), turned to 180 degrees
- moved JP3 67.1 mm to (23.4, 22.0)
- moved C87 66.5 mm to (36.3, 22.9), turned to 90 degrees
- moved D25 59.8 mm to (29.8, 35.8), turned to 0 degrees
- moved D26 58.2 mm to (29.8, 34.0), turned to 180 degrees
- moved ZD1 57.3 mm to (28.1, 26.0), turned to 270 degrees
- moved R57 56.2 mm to (52.0, 76.9), turned to 180 degrees
- moved D24 54.0 mm to (31.8, 22.0), turned to 90 degrees
- moved D23 52.2 mm to (27.8, 30.9)
- moved IC21 36.4 mm to (45.4, 79.6), turned to 0 degrees
- moved R56 33.2 mm to (52.9, 85.8), turned to 180 degrees
- moved R59 22.1 mm to (22.4, 19.7), turned to 0 degrees
- moved R63 11.9 mm to (36.8, 41.1), turned to 270 degrees
- moved R58 9.33 mm to (22.4, 29.1)
- moved R65 6.71 mm to (39.6, 31.2)
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Connections:
- removed net ADIB1N: JP2.2, K1.2, X5.3
- removed net ADIB1P: JP3.2, K1.9, X5.4
- removed net ADIB1_R: IC21.5, IC8.101
- removed net ADIB1_S: IC21.2, IC8.117
- removed net ADIB2N: JP4.2, K2.2, X6.3
- removed net ADIB2P: JP5.2, K2.9, X6.4
- removed net ADIB2_R: IC21.12, IC8.103
- removed net ADIB2_S: IC21.9, IC8.102
- removed net N$28: D24.A, IC21.6, K1.5
- removed net N$33: D23.C, D24.C, D25.C, D26.C, ZD1.C
- removed net N$40: D25.A, IC21.8, K2.6
- removed net N$41: D26.A, IC21.11, K2.5
- new net ADIB1_SW: IC21.1, IC21.16, IC8.117
- new net ADIB2_SW: IC21.8, IC21.9, IC8.102
- net +15V_ISO: now also IC21.13, R60.1; no longer R59.1
- net +3V3_ISO: now also C87.2; no longer C88.2
- net +5V_ISO: now also IC21.12; no longer C87.2, IC21.14, K1.1, K1.10, K2.1, K2.10, R56.1, ZD1.A
- net -15V_ISO: now also IC21.4, R66.1; no longer R65.1
- net -VSENSE: now also IC21.2, IC21.7; no longer JP2.3, JP4.1, K1.4, K2.4
- net AFE1N: now also IC21.3, X5.3; no longer JP2.1, K1.3
- net AFE1P: now also R56.1, X5.4; no longer JP3.3, K1.8
- net AFE2N: now also IC21.6, X6.3; no longer JP4.3, K2.3
- net AFE2P: now also R57.1, X6.4; no longer JP5.1, K2.8
- net BIAS_EN: now also R63.1; no longer R62.1
- net CLAMP: now also D23.2, D24.2; no longer D27.2, D28.2
- net DAC_OUT#1: now also IC21.15; no longer JP3.1, K1.7
- net DAC_OUT#2: now also IC21.10; no longer JP5.3, K2.7
- net GND: now also D23.1, D24.1, IC21.5, ZD1.A, ZD2.C; no longer C88.1, D27.1, D28.1, IC21.7, ZD2.A, ZD3.C
- net N$129: now also D23.3, R58.2; no longer D27.3, R57.2
- net N$134: now also D24.3, R59.2; no longer D28.3, R58.2
- net N$149: now also R62.2; no longer R61.2
- net N$151: now also R61.2, R62.1; no longer R60.2, R61.1
- net N$152: now also D25.A; no longer D29.A
- net N$153: now also D25.C, JP2.3, ZD1.C; no longer D29.C, JP6.3, ZD2.C
- net N$154: now also R60.2, R61.1; no longer R59.2, R60.1
- net N$155: now also R64.2, R65.1; no longer R63.2, R64.1
- net N$162: now also R66.2; no longer R64.2
- net N$163: now also R64.1; no longer R63.1
- net N$164: now also D26.C; no longer D30.C
- net N$168: now also D26.A, JP3.3, ZD2.A; no longer D30.A, JP7.3, ZD3.A
- net N$20: now also IC21.14; no longer IC21.1, IC21.10, IC21.13, IC21.4
- net N$22: now also IC21.11, R57.2; no longer D23.A, IC21.3, K1.6
- net N$25: now also JP2.2; no longer JP6.2
- net N$3: now also R63.2; no longer R62.2
- net N$39: now also JP3.2; no longer JP7.2
- net N$4: now also JP2.1, R58.1; no longer JP6.1, R57.1
- net N$6: now also JP3.1, R59.1; no longer JP7.1, R58.1
Routing:
- net ADIB2_SW: track 0.00 -> 86.9 mm, vias 0 -> 2
- net ADIB1_SW: track 0.00 -> 79.8 mm, vias 0 -> 4
- net ADIB2_R: track 60.9 -> 0.00 mm, vias 4 -> 0
- net +5V_ISO: track 255.3 -> 207.1 mm, vias 9 -> 7
- net ADIB1_R: track 48.1 -> 0.00 mm, vias 2 -> 0
- net -VSENSE: track 260.8 -> 213.2 mm, vias 7 -> 4
- net ADIB2_S: track 46.3 -> 0.00 mm, vias 2 -> 0
- net ADIB2P: track 45.3 -> 0.00 mm
- net ADIB1_S: track 43.2 -> 0.00 mm, vias 4 -> 0
- net N$28: track 38.3 -> 0.00 mm
- net N$22: track 39.8 -> 3.33 mm, vias 2 -> 0
- net ADIB1N: track 33.5 -> 0.00 mm
- net ADIB2N: track 28.1 -> 0.00 mm
- net DAC_OUT#2: track 162.5 -> 135.3 mm, vias 5 -> 4
- net N$33: track 24.5 -> 0.00 mm, vias 3 -> 0
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Other:
- board text added: "EEZ DIB MIO168 (04/2021 r2B5)"
- board text added: "EEZ DIB MIO168 (04/2021 r2B5) Project source code: github.com/eez-open"
- board text removed: "EEZ DIB MIO168 (01/2021 r2B4)"
- board text removed: "EEZ DIB MIO168 (01/2021 r2B4) Project source code: github.com/eez-open"
