File: EDA files/EEZ DIB MIO168 r2B5.brd (EAGLE design)
At the start: 146 x 95 mm, 255 parts, among them IC1 M24C32-WMN6P, IC10 OPA2196IDR, IC11 DAC7760IPWPR, IC12 DAC7760IPWPR, IC13 OPA376AIDBVR, IC14 DAC7563TDGSR, IC15 OPA2196IDR, IC16 BTS3408G, IC17 BTS3408G, IC18 BTS3408G, IC19 BTS3408G, IC2 Si8641BB-B-IS1, IC20 TL431B, IC21 DG212BDY-T1-E3, IC22 74HC126PW,118, IC3 Si8641BB-B-IS1, IC4 LP2985-33DBVR, IC5 L78L15, IC6 SN6505BDBVT, IC7 L79L15, IC8 STM32F446ZCT6, IC9 N.C., J1 4907, J2 N.C., Q1 2N7002PS,115, Q10 MMBT5551, Q11 2N7002, Q2 2N7002PS,115, Q3 2N7002PS,115, Q4 2N7002PS,115, Q5 2N7002PS,115, Q6 BSS84P, Q7 MMBT5401, Q8 BSS84P, Q9 MMBT5551, X1 77317-104-28LF, X2 N.C., X3 691327310016, X4 691322310008, X5 DS1014-10RF1B, X6 DS1014-10RF1B, X7 DS1023-2*14S21, X8 DS1023-2*14S21, Y1 LF XTAL026392

Commit message: BOM update
Parts:
- added C88, C89: N.C., rcl:C0805
- moved R32 10.9 mm to (11.7, 77.0)
- moved R33 10.9 mm to (11.7, 73.3)
- moved R34 10.9 mm to (11.7, 69.6)
- moved R35 10.9 mm to (11.7, 65.9)
- moved R36 10.9 mm to (11.7, 62.2)
- moved R37 10.9 mm to (11.7, 58.5)
- moved R38 10.9 mm to (11.7, 54.9)
- moved R39 10.9 mm to (11.7, 51.2)
- moved TVS4 3.54 mm to (44.9, 42.2), turned to 90 degrees
- moved TVS3 2.59 mm to (47.1, 53.4), turned to 270 degrees
- moved R14 1.97 mm to (47.1, 47.2)
- moved R15 1.97 mm to (49.1, 47.2)
- moved R25 1.97 mm to (47.1, 43.3)
- moved R24 1.97 mm to (49.1, 43.3)
Connections:
- net N$55: now also C88.1
- net N$56: now also C88.2
- net N$58: now also C89.1
- net N$59: now also C89.2
Routing:
- net DIN7/MISO: track 120.7 -> 131.6 mm
- net DIN1: track 97.6 -> 108.5 mm
- net N$42: track 16.0 -> 5.07 mm
- net N$36: track 16.2 -> 5.23 mm
- net N$120: track 15.8 -> 4.86 mm
- net N$119: track 15.8 -> 4.92 mm
- net N$109: track 15.9 -> 5.02 mm
- net N$38: track 16.0 -> 5.13 mm
- net N$14: track 16.1 -> 5.18 mm
- net N$122: track 15.9 -> 4.97 mm
- net DIN5: track 89.6 -> 100.5 mm
- net DIN4: track 89.7 -> 100.6 mm
- net DIN3: track 93.0 -> 103.9 mm
- net DIN2: track 96.0 -> 106.9 mm
- net DIN0: track 100.4 -> 111.3 mm
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Other:
- board text added: "EEZ DIB MIO168 (07/2021 r2B5)"
- board text added: "EEZ DIB MIO168 (07/2021 r2B5) Project source code: github.com/eez-open"
- board text removed: "EEZ DIB MIO168 (06/2021 r2B5)"
- board text removed: "EEZ DIB MIO168 (06/2021 r2B5) Project source code: github.com/eez-open"
