File: EDA files/EEZ DIB MIO168 r2B5.sch (EAGLE design)
At the start: 265 parts, among them IC1 M24C32-WMN6P, IC10 OPA2196IDR, IC11 DAC7760IPWPR, IC12 DAC7760IPWPR, IC13 OPA376AIDBVR, IC14 DAC7563TDGSR, IC15 OPA2196IDR, IC16 BTS3408G, IC17 BTS3408G, IC18 BTS3408G, IC19 BTS3408G, IC2 Si8641BB-B-IS1, IC20 TL431B, IC21 74HC126PW,118, IC22 74HC126PW,118, IC3 Si8641BB-B-IS1, IC4 LP2985-33DBVR, IC5 L78L15, IC6 SN6505BDBVT, IC7 L79L15, IC8 STM32F446ZCT6, IC9 N.C., J1 4907, J2 N.C., K1 TQ2SS-L2-5V-X, K2 TQ2SS-L2-5V-X, Q1 2N7002PS,115, Q10 MMBT5551, Q11 2N7002, Q2 2N7002PS,115, Q3 2N7002PS,115, Q4 2N7002PS,115, Q5 2N7002PS,115, Q6 BSS84P, Q7 MMBT5401, Q8 BSS84P, Q9 MMBT5551, X1 77317-104-28LF, X2 N.C., X3 691327310016, X4 691322310008, X5 DS1014-10RF1B, X6 DS1014-10RF1B, X7 DS1023-2*14S21, X8 DS1023-2*14S21, Y1 LF XTAL026392

Commit message: r2B5, ADIB switcing
Parts:
- removed C88: 100n, rcl:C-EUC0603
- removed D27, D28: BAT54SFILM, diode:BAT54S
- removed D29, D30: MBR0530T3G, EEZ_Lib1:SCHOTTKYSOD123
- removed JP4, JP5, JP6, JP7: DS1025-01-1*3P8BV1-B, EEZ_connectors:JUMPER-3PIN2MM
- removed K1, K2: TQ2SS-L2-5V-X, EEZ_switches:TQ2SS-L2RELAY_TQ2_SS_PAN-M
- removed ZD3: SMAJ16A, EEZ_Lib1:SMAJ-ADO214AC
- added R66: 47R, rcl:R-EU_R0805
- C1: value 100n -> N.C.
- D23, D24: value BAS316 -> BAT54SFILM; device EEZ_Lib1:DIODESOD323R -> diode:BAT54S
- D25, D26: value BAS316 -> MBR0530T3G; device EEZ_Lib1:DIODESOD323R -> EEZ_Lib1:SCHOTTKYSOD123
- IC21: value 74HC126PW,118 -> DG212BDY-T1-E3; device EEZ_DIB:74HC126PW,118 -> EEZ_DIB:DG212BDY-T1-E3
- R56: value 100K -> 1K
- R57: value 100R -> 1K
- R59: value 47R -> 100R
- R60: value 100K -> 47R
- R61: value 10K -> 100K
- R62: value 470R -> 10K
- R63: value 10K -> 470R
- R64: value 100K -> 10K
- R65: value 47R -> 100K
- ZD1: value MM3Z18VT1G -> SMAJ16A; device EEZ_Lib1:ZENER-DIODESOD323R -> EEZ_Lib1:SMAJ-ADO214AC
Connections:
- removed net ADIB1N: JP2.2, K1G$2.NC, X5-3.1
- removed net ADIB1P: JP3.2, K1G$3.NC, X5-4.1
- removed net ADIB1_R: IC21B.I, IC8A.PA9
- removed net ADIB1_S: IC21A.I, IC8A.PD3
- removed net ADIB2N: JP4.2, K2G$2.NC, X6-3.1
- removed net ADIB2P: JP5.2, K2G$3.NC, X6-4.1
- removed net ADIB2_R: IC21D.I, IC8A.PA11
- removed net ADIB2_S: IC21C.I, IC8A.PA10
- removed net N$28: D24.A, IC21B.O, K1G$1.R-
- removed net N$33: D23.C, D24.C, D25.C, D26.C, ZD1.C
- removed net N$40: D25.A, IC21C.O, K2G$1.S-
- removed net N$41: D26.A, IC21D.O, K2G$1.R-
- new net ADIB1_SW: IC21A.IN, IC21B.IN, IC8A.PD3
- new net ADIB2_SW: IC21C.IN, IC21D.IN, IC8A.PA10
- net +15V_ISO: now also IC21P.V+, R60.1; no longer R59.1
- net +3V3_ISO: now also C87.2; no longer C88.2
- net +5V_ISO: now also IC21P.VL; no longer C87.2, IC21P.V+, K1G$1.R+, K1G$1.S+, K2G$1.R+, K2G$1.S+, R56.1, ZD1.A
- net -15V_ISO: now also IC21P.V-, R66.1; no longer R65.1
- net -VSENSE: now also IC21A.D, IC21D.D; no longer JP2.3, JP4.1, K1G$2.NO, K2G$2.NO
- net AFE1N: now also IC21A.S, X5-3.1; no longer JP2.1, K1G$2.COM
- net AFE1P: now also R56.1, X5-4.1; no longer JP3.3, K1G$3.COM
- net AFE2N: now also IC21D.S, X6-3.1; no longer JP4.3, K2G$2.COM
- net AFE2P: now also R57.1, X6-4.1; no longer JP5.1, K2G$3.COM
- net BIAS_EN: now also R63.1; no longer R62.1
- net CLAMP: now also D23.C2, D24.C2; no longer D27.C2, D28.C2
- net DAC_OUT#1: now also IC21B.D; no longer JP3.1, K1G$3.NO
- net DAC_OUT#2: now also IC21C.D; no longer JP5.3, K2G$3.NO
- net GND: now also D23.A1, D24.A1, IC21P.GND, ZD1.A, ZD2.C; no longer C88.1, D27.A1, D28.A1, IC21P.V-, ZD2.A, ZD3.C
- net N$129: now also D23.C1A2, R58.2; no longer D27.C1A2, R57.2
- net N$134: now also D24.C1A2, R59.2; no longer D28.C1A2, R58.2
- net N$149: now also R62.2; no longer R61.2
- net N$151: now also R61.2, R62.1; no longer R60.2, R61.1
- net N$152: now also D25.A; no longer D29.A
- net N$153: now also D25.C, JP2.3, ZD1.C; no longer D29.C, JP6.3, ZD2.C
- net N$154: now also R60.2, R61.1; no longer R59.2, R60.1
- net N$155: now also R64.2, R65.1; no longer R63.2, R64.1
- net N$162: now also R66.2; no longer R64.2
- net N$163: now also R64.1; no longer R63.1
- net N$164: now also D26.C; no longer D30.C
- net N$168: now also D26.A, JP3.3, ZD2.A; no longer D30.A, JP7.3, ZD3.A
- net N$20: now also IC21B.S; no longer IC21A.EN, IC21B.EN, IC21C.EN, IC21D.EN
- net N$22: now also IC21C.S, R57.2; no longer D23.A, IC21A.O, K1G$1.S-
- net N$25: now also JP2.2; no longer JP6.2
- net N$3: now also R63.2; no longer R62.2
- net N$39: now also JP3.2; no longer JP7.2
- net N$4: now also JP2.1, R58.1; no longer JP6.1, R57.1
- net N$6: now also JP3.1, R59.1; no longer JP7.1, R58.1
Other:
- note added: "ADIB switches and AFE connectors PWM outputs / sensor bias"
- note removed: "PWM outputs / sensor bias ADIB and AFE connectors"
- moved on the sheet: C87, JP2, JP3, R56, R57, R58, R59, R60, R61, R62, R63, R64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
