File: EDA files/EEZ DIB MIO168 r2B5.sch (EAGLE design)
At the start: 254 parts, among them IC1 M24C32-WMN6P, IC10 OPA2196IDR, IC11 DAC7760IPWPR, IC12 DAC7760IPWPR, IC13 OPA376AIDBVR, IC14 DAC7563TDGSR, IC15 OPA2196IDR, IC16 BTS3408G, IC17 BTS3408G, IC18 BTS3408G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

Commit message: BOM update
Parts:
- added C88, C89: N.C., rcl:C-EUC0805
Connections:
- net N$55: now also C88.1
- net N$56: now also C88.2
- net N$58: now also C89.1
- net N$59: now also C89.2
Other:
- moved on the sheet: C63, C64, C65, C66, C67, C68, C69, C70, D13, D14, IC13A, IC13P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
